File: BRAUNIT Charging Dock.kicad_pcb (KiCad board)
At the start: 2 copper layers, 65 x 45 mm, 69 parts, among them J1 BRAUNIT, J2 BRAUNIT, J3 TYPE-C-31-M-12, J4 BM04B-SRSS-TB, Q1 AO4459, Q2 2N7002, Q3 AO4459, Q4 2N7002, Q5 AO4459, Q6 2N7002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

Commit message: WIP traces
Parts:
- added JP1: SolderJumper_2_Open, Jumper:SolderJumper-2_P1.3mm_Open_TrianglePad1.0x1.5mm, B.Cu at (178.7, 74.5)
- moved D14 42.5 mm to (148.6, 109.8), turned to 180 degrees
- moved R16 37.7 mm to (147.5, 108.2)
- moved R17 37.7 mm to (147.5, 106.7)
- moved D12 7.03 mm to (149.4, 92.9), turned to 0 degrees
- moved J4 1.78 mm to (160.5, 69.1)
- moved R14 0.51 mm to (153.7, 77.3)
- moved C17 0.40 mm to (153.2, 88.6)
- moved R15 0.25 mm to (153.7, 79.1)
- moved R13 0.25 mm to (154.1, 86.0)
- moved locked 0.25 mm to (149.7, 83.7)
- renumbered R12 to locked
Routing:
- net VCC: track 0.00 -> 111.9 mm
- net EN_R: track 0.00 -> 78.6 mm, vias 0 -> 3
- net GND: track 0.00 -> 42.8 mm, vias 0 -> 19
- net VDD: track 0.00 -> 42.3 mm
- net Net-(C18-Pad2): track 0.00 -> 37.7 mm, vias 0 -> 9
- net Net-(R17-Pad2): track 0.00 -> 31.3 mm, vias 0 -> 2
- net Net-(J4-Pad3): track 0.00 -> 14.6 mm
- net Net-(J4-Pad4): track 0.00 -> 12.8 mm
- net Net-(Q5-Pad4): track 0.00 -> 6.82 mm
- net Net-(R9-Pad2): track 0.00 -> 6.38 mm
- net Net-(D10-Pad1): track 0.00 -> 6.29 mm
- net Net-(D9-Pad1): track 0.00 -> 6.10 mm
- net Net-(C16-Pad1): track 0.00 -> 5.28 mm
- net unconnected-(J4-PadMP): track 0.00 -> 5.00 mm
- net Net-(C15-Pad1): track 0.00 -> 4.70 mm
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- added copper zone on B.Cu, net GND
- added copper zone on F.Cu, net GND
- added copper zone on B.Cu, net Net-(C18-Pad2)
- added copper zone on B.Cu, net VCC

Commit message: Change to 4-layer board and do some routing
Parts:
- added H1: MountingHole, BRAUNIT Charger:MountingHole_2.7mm_M2.5_DIN912_Keepout, F.Cu at (118.3, 68.7)
- added H2: MountingHole, BRAUNIT Charger:MountingHole_2.7mm_M2.5_DIN912_Keepout, F.Cu at (178.8, 68.7)
- added H3: MountingHole, BRAUNIT Charger:MountingHole_2.7mm_M2.5_DIN912_Keepout, F.Cu at (118.3, 109.2)
- added H4: MountingHole, BRAUNIT Charger:MountingHole_2.7mm_M2.5_DIN912_Keepout, F.Cu at (178.8, 109.2)
- added H5: MountingHole, BRAUNIT Charger:MountingHole_2.7mm_M2.5_DIN912_Keepout, F.Cu at (148.6, 96.4)
- moved C17 3.43 mm to (155.3, 86.0), turned to 90 degrees
- moved R2 2.90 mm to (133.2, 107.4), turned to 90 degrees
- moved R6 2.90 mm to (165.7, 107.4), turned to 90 degrees
- moved R17 2.17 mm to (149.5, 107.4), turned to 90 degrees
- moved R1 1.27 mm to (131.5, 107.4), turned to 90 degrees
- moved R5 1.27 mm to (164.0, 107.4), turned to 90 degrees
- moved R16 0.80 mm to (147.7, 107.4), turned to 90 degrees
- moved R14 0.51 mm to (153.7, 77.8)
- moved R9 0.38 mm to (144.9, 86.3)
- moved R15 0.25 mm to (153.7, 79.4)
- moved R13 0.25 mm to (153.8, 86.0)
- renumbered D9 to locked
Routing:
- net VCC: track 111.9 -> 73.1 mm
- net Net-(C18-Pad2): track 37.7 -> 17.2 mm, vias 9 -> 10
- net GND: track 42.8 -> 62.1 mm, vias 19 -> 43
- net /Charger Right/NTC: track 0.00 -> 16.3 mm, vias 0 -> 1
- net /Charger Left/NTC: track 0.00 -> 15.1 mm, vias 0 -> 1
- net VDD: track 42.3 -> 28.4 mm, vias 0 -> 2
- net /Charger Right/EN: track 1.74 -> 14.9 mm, vias 0 -> 1
- net /Charger Left/EN: track 1.72 -> 14.8 mm, vias 0 -> 1
- net EN_R: track 78.6 -> 65.5 mm
- net Net-(R17-Pad2): track 31.3 -> 33.6 mm
- net Net-(D7-Pad4): track 0.00 -> 1.91 mm
- net Net-(D3-Pad4): track 0.00 -> 1.90 mm
- net Net-(D14-Pad1): track 3.32 -> 1.55 mm
- net Net-(D7-Pad3): track 0.00 -> 1.77 mm
- net Net-(D3-Pad3): track 0.00 -> 1.76 mm
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Other:
- copper layers 2 -> 4

Commit message: Only output connections to go :)
Parts:
- NT1, NT2: moved to F.Cu
- moved NT1 35.6 mm to (141.6, 68.1), turned to 0 degrees
- moved NT2 32.1 mm to (155.6, 68.1), turned to 180 degrees
- moved C11 23.7 mm to (173.1, 77.4), turned to 90 degrees
- moved C9 23.1 mm to (175.4, 76.7), turned to 180 degrees
- moved C4 22.2 mm to (124.1, 98.8), turned to -90 degrees
- moved C2 21.6 mm to (121.8, 99.5), turned to 0 degrees
- moved R8 21.1 mm to (175.4, 78.2), turned to 180 degrees
- moved R4 19.7 mm to (121.8, 98.0), turned to 0 degrees
- moved R9 0.38 mm to (144.9, 86.0)
Routing:
- net VCC: track 73.1 -> 138.3 mm
- net Net-(C2-Pad2): track 0.00 -> 54.7 mm, vias 0 -> 3
- net Net-(C10-Pad2): track 0.00 -> 41.7 mm, vias 0 -> 3
- net Net-(C18-Pad2): track 17.2 -> 53.3 mm, vias 10 -> 8
- net Net-(R5-Pad2): track 1.23 -> 35.2 mm, vias 1 -> 2
- net Net-(R6-Pad2): track 1.23 -> 33.4 mm, vias 1 -> 2
- net Net-(R1-Pad2): track 1.23 -> 23.3 mm, vias 1 -> 2
- net Net-(R2-Pad2): track 1.23 -> 22.6 mm, vias 1 -> 2
- net Net-(C9-Pad1): track 0.00 -> 16.3 mm, vias 0 -> 2
- net Net-(R8-Pad1): track 0.00 -> 16.2 mm, vias 0 -> 2
- net Net-(R4-Pad1): track 0.00 -> 14.7 mm, vias 0 -> 2
- net Net-(C2-Pad1): track 0.00 -> 14.7 mm, vias 0 -> 2
- net Net-(Rcs2-Pad3): track 0.00 -> 13.0 mm
- net Net-(Rcs1-Pad3): track 0.00 -> 13.0 mm
- net Net-(Rcs1-Pad2): track 0.00 -> 10.1 mm
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- added copper zone on B.Cu, net Net-(D1-Pad1)
- added copper zone on B.Cu, net Net-(D1-Pad2)
- added copper zone on B.Cu, net Net-(D5-Pad1)
- added copper zone on B.Cu, net Net-(D5-Pad2)
- added copper zone on B.Cu, net Net-(L1-Pad2)
- added copper zone on B.Cu, net Net-(L2-Pad2)
